File: 2s 40A PSU and charger.kicad_pcb (KiCad board)
At the start: 4 copper layers, 45 x 20 mm, 115 parts, among them J1 Keystone 6100, J10 G-Switch-GT-USB-7025, J12 USB, J13 Precidip 853-87-004-20-001101, J2 JST XH-S Balance Plug, J3 Keystone 6100, J4 Keystone 6102, J5 Keystone 6102, J6 Keystone 6100, J7 Keystone 6100, J8 Keystone 6102, J9 Keystone 6102, Q1 PJA3430, or HL 2320A, Q2 PJA3430, or HL 2320A, Q3 Vishay sir404dp, or SiR500DP, Q4 PJA3430, or HL 2320A, Q5 PJA3430, or HL 2320A, Q6 Vishay sir404dp, or SiR500DP, SW1 Mitsumi R-667996, U1 BQ76905RGRR, U2 AP63203WU, U3 BQ24780SRUYR, U5 THVD1420DRLR, U6 CH32X035G8U6, U7 TPS7A2633DRV

Commit message: Finished design & silk
Other:
- board text added: "- +"
- board text added: "D-D+"
- board text removed: "+ D+D- -"

Commit message: Replaced inductor value and lcsc part
Parts:
- L3: value 2.7uH -> 3.3uH
Changed lines of the file:
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@@
 			)
 		)
-		(property "Value" "2.7uH"
+		(property "Value" "3.3uH"
 			(at -0.2 1.7 90)
 			(layer "B.Fab")
@@
 			)
 		)
-		(property "LCSC" ""
+		(property "LCSC" "C2041573"
 			(at 0 0 270)
 			(unlocked yes)
